File: Hardware/Haptic_Motor_Driver_DRV2605L.brd (EAGLE design)
At the start: 20.3 x 21.6 mm, 15 parts, among them U1 DRV2605L

Commit message: Updated BRD files per EDR
Parts:
- moved FRAME2 5.39 mm to (-12.7, -14.0)
- moved FID1 1.36 mm to (6.35, 1.27)
- moved FID2 1.27 mm to (18.9, 13.8)
- moved LOGO4 1.27 mm to (18.0, 9.56)
- moved JP1 1.27 mm to (1.27, 1.27)
- moved C1 1.27 mm to (12.5, 14.6)
- moved C3 1.27 mm to (7.94, 14.6)
- moved I2C 1.27 mm to (11.0, 6.83)
- moved JP2 1.27 mm to (19.1, 8.89)
- moved R1 1.27 mm to (13.8, 6.67)
- moved R2 1.27 mm to (7.94, 6.67)
- moved STANDOFF1 1.27 mm to (17.8, 17.8)
- moved STANDOFF4 1.27 mm to (2.54, 17.8)
- moved U1 1.27 mm to (10.6, 11.7)
Other:
- board size 20.3 x 21.6 mm -> 20.3 x 20.3 mm
- board text added: "0x5A"
