File: Hardware/Haptic_Motor_Driver_DRV2605L.brd (EAGLE design)
At the start: 20.3 x 20.3 mm, 15 parts, among them U1 DRV2605L

Commit message: Updated Silk
Other:
- board text added: "I2C ADDR 0x5A"
- board text added: "I2C PU"
- board text removed: "0x5A"
- board text removed: "I2C"
